Commit message: Adding Lidar

File: description/robot.urdf.xacro (robot description, xacro)
@@ -3,3 +3,4 @@
     <xacro:include filename="robot_core.xacro"/>
     <xacro:include filename="gazebo_control.xacro"/>
+    <xacro:include filename="lidar.xacro"/>
 </robot>

File: description/robot_core.xacro (robot description, xacro)
@@ -9,8 +9,11 @@
     </material>
     <material name= "orange">
-        <color rgba="1 0 0 1"/>
+        <color rgba="1 0.3 0.1 1"/>
     </material>
     <material name= "green">
         <color rgba="0 1 0 1"/>
+    </material>
+    <material name= "red">
+        <color rgba="1 0 0 1"/>
     </material>
     <!-- BASE LINK -->
